File: lumberjack.kicad_pcb (KiCad board)
At the start: 2 copper layers, 424.7 x 94.2 mm, 199 parts, among them J1 USB, J2 AVR_ISP_6, J3 JST, J4 JST, SW1 RESET, SW2 BOOT, U1 ATMEGA328-PU, Y1 16MHz

Commit message: layout new switches and diodes
Parts:
- moved 2u_MX60 460.7 mm to (76.2, 179.1)
- moved 2u_MX30 328.3 mm to (218.4, 179.1)
- moved D40 239.5 mm to (149.9, 145.0), turned to 90 degrees
- moved D66 232.5 mm to (181.6, 137.8), turned to 180 degrees
- moved D65 222.0 mm to (181.6, 127.6), turned to 180 degrees
- moved D71 218.2 mm to (189.2, 142.9)
- moved D34 213.0 mm to (167.2, 126.7), turned to -90 degrees
- moved D33 210.5 mm to (191.8, 127.6)
- moved D67 209.8 mm to (181.6, 117.5), turned to 180 degrees
- moved D72 209.7 mm to (160.5, 126.7), turned to -90 degrees
- moved D39 206.6 mm to (191.8, 137.8)
- moved D78 196.0 mm to (164.1, 126.7), turned to -90 degrees
- moved D82 190.9 mm to (191.8, 97.2)
- moved D80 188.4 mm to (179.1, 102.2), turned to 180 degrees
- moved D77 188.2 mm to (189.2, 132.7)
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Routing:
- net /COL7: track 0.00 -> 215.3 mm
- net /COL1: track 0.00 -> 104.3 mm
- net /COL4: track 0.00 -> 96.9 mm
- net /COL9: track 0.00 -> 95.3 mm
- net /COL3: track 0.00 -> 95.3 mm
- net /COL2: track 0.00 -> 95.3 mm
- net /COL0: track 5.39 -> 98.5 mm
- net /COL6: track 0.00 -> 87.7 mm
- net /COL8: track 0.00 -> 57.2 mm
- net Net-(D76-A): vias 0 -> 1
- net GND: vias 19 -> 17
- net /ROW3: vias 0 -> 1
Other:
- board size 424.7 x 94.2 mm -> 404.3 x 94.2 mm

Commit message: new IC and updated col layout
Parts:
- removed 2u_MX30, 2u_MX60: SW_Push, lumberjack:MX_PCB_200B
- removed U1: ATMEGA328-PU, Package_DIP:DIP-28_W7.62mm
- added U2: ATmega32A-P, Package_DIP:DIP-40_W15.24mm, F.Cu at (153.1, 69.6)
- D61, D62: value 3.6V -> 1N4148
- D81, D82: value 1N4148 -> 3.6V
- MX7: footprint lumberjack:MX -> lumberjack:MX_NTHSTH
- MX8: footprint lumberjack:MX_NTHSTH -> lumberjack:MX
- moved MX57 195.3 mm to (268.9, 83.3)
- moved MX58 195.3 mm to (268.9, 102.4)
- moved MX59 195.3 mm to (268.9, 121.4)
- moved MX56 195.1 mm to (268.8, 64.3)
- moved MX60 195.1 mm to (268.8, 140.5)
- moved MX31 176.2 mm to (73.7, 64.3)
- moved MX32 176.2 mm to (73.7, 83.3)
- moved MX33 176.2 mm to (73.7, 102.4)
- moved MX34 176.2 mm to (73.7, 121.4)
- moved MX35 176.2 mm to (73.7, 140.5)
- moved MX55 174.7 mm to (249.9, 140.5)
- moved MX51 158.3 mm to (249.9, 64.3)
- moved MX52 158.3 mm to (249.9, 83.3)
- moved MX53 158.3 mm to (249.9, 102.4)
- moved MX54 158.3 mm to (249.9, 121.4)
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Connections:
- net /RESET renamed Net-(J2-Pin_2)
- D10 pad 1: /ROW3 -> /ROW4
- D11 pad 1: /ROW4 -> /ROW0
- D13 pad 1: /ROW0 -> /ROW2
- D14 pad 1: /ROW1 -> /ROW3
- D15 pad 1: /ROW2 -> /ROW4
- D16 pad 1: /ROW3 -> /ROW0
- D17 pad 1: /ROW4 -> /ROW1
- D18 pad 1: /ROW1 -> /ROW2
- D19 pad 1: /ROW0 -> /ROW3
- D20 pad 1: /ROW1 -> /ROW4
- D21 pad 1: /ROW2 -> /ROW0
- D22 pad 1: /ROW3 -> /ROW1
- D23 pad 1: /ROW4 -> /ROW2
- D24 pad 1: /ROW1 -> /ROW3
- D25 pad 1: /ROW0 -> /ROW4
- D26 pad 1: /ROW1 -> /ROW0
- D27 pad 1: /ROW2 -> /ROW1
- D28 pad 1: /ROW3 -> /ROW2
- D29 pad 1: /ROW4 -> /ROW3
- D30 pad 1: /ROW1 -> /ROW4
- D36 pad 1: /ROW1 -> /ROW0
- D37 pad 1: /ROW0 -> /ROW1
- D38 pad 1: /ROW1 -> /ROW2
- D39 pad 1: /ROW2 -> /ROW3
- D40 pad 1: /ROW3 -> /ROW4
- D41 pad 1: /ROW4 -> /ROW0
- D43 pad 1: /ROW0 -> /ROW2
- D44 pad 1: /ROW1 -> /ROW3
- D45 pad 1: /ROW2 -> /ROW4
- D46 pad 1: /ROW3 -> /ROW0
- D47 pad 1: /ROW4 -> /ROW1
- D48 pad 1: /ROW1 -> /ROW2
- D49 pad 1: /ROW0 -> /ROW3
- D50 pad 1: /ROW1 -> /ROW4
- D51 pad 1: /ROW2 -> /ROW0
- D52 pad 1: /ROW3 -> /ROW1
- D53 pad 1: /ROW4 -> /ROW2
- D54 pad 1: /ROW1 -> /ROW3
- D55 pad 1: /ROW0 -> /ROW4
- D56 pad 1: /ROW1 -> /ROW0
- D57 pad 1: /ROW2 -> /ROW1
- D58 pad 1: /ROW3 -> /ROW2
- D59 pad 1: /ROW4 -> /ROW3
- D6 pad 1: /ROW1 -> /ROW0
- D60 pad 1: /ROW1 -> /ROW4
- D61 pad 1: Net-(D61-K) -> /ROW0
- D61 pad 2: GND -> Net-(D61-A)
- D62 pad 1: Net-(D62-K) -> /ROW1
- D62 pad 2: GND -> Net-(D62-A)
- D63 pad 1: /ROW0 -> /ROW2
- D64 pad 1: /ROW1 -> /ROW3
- D65 pad 1: /ROW2 -> /ROW4
- D66 pad 1: /ROW3 -> /ROW0
- D67 pad 1: /ROW4 -> /ROW1
- D68 pad 1: /ROW1 -> /ROW2
- D69 pad 1: /ROW0 -> /ROW3
- D7 pad 1: /ROW0 -> /ROW1
- D70 pad 1: /ROW1 -> /ROW4
- D71 pad 1: /ROW2 -> /ROW0
- D72 pad 1: /ROW3 -> /ROW1
- D73 pad 1: /ROW4 -> /ROW2
- D74 pad 1: /ROW1 -> /ROW3
- D75 pad 1: /ROW0 -> /ROW4
- D76 pad 1: /ROW1 -> /ROW0
- D77 pad 1: /ROW2 -> /ROW1
- D78 pad 1: /ROW3 -> /ROW2
- D79 pad 1: /ROW4 -> /ROW3
- D8 pad 1: /ROW1 -> /ROW2
- D80 pad 1: /ROW1 -> /ROW4
- D81 pad 1: /ROW0 -> Net-(D81-K)
- D81 pad 2: Net-(D81-A) -> GND
- D82 pad 1: /ROW1 -> Net-(D82-K)
- D82 pad 2: Net-(D82-A) -> GND
- D9 pad 1: /ROW2 -> /ROW3
- J1 pad A6: Net-(D61-K) -> Net-(D81-K)
- J1 pad A7: Net-(D62-K) -> Net-(D82-K)
- J1 pad B6: Net-(D61-K) -> Net-(D81-K)
- J1 pad B7: Net-(D62-K) -> Net-(D82-K)
- J3 pad 2: Net-(D62-K) -> Net-(D82-K)
- J3 pad 3: Net-(D61-K) -> Net-(D81-K)
- J4 pad 2: Net-(D61-K) -> Net-(D81-K)
- J4 pad 3: Net-(D62-K) -> Net-(D82-K)
- MX11 pad 2: /COL1 -> /COL2
- MX12 pad 2: /COL1 -> /COL2
- MX16 pad 2: /COL2 -> /COL3
- MX17 pad 2: /COL2 -> /COL3
- MX18 pad 2: /COL2 -> /COL3
- MX21 pad 2: /COL3 -> /COL4
- MX22 pad 2: /COL3 -> /COL4
- MX23 pad 2: /COL3 -> /COL4
- MX24 pad 2: /COL3 -> /COL4
- MX26 pad 2: /COL4 -> /COL5
- MX27 pad 2: /COL4 -> /COL5
- MX28 pad 2: /COL4 -> /COL5
- MX29 pad 2: /COL4 -> /COL5
- MX30 pad 2: /COL4 -> /COL5
- MX31 pad 2: /COL5 -> /COL6
- MX32 pad 2: /COL5 -> /COL6
- MX33 pad 2: /COL5 -> /COL6
- MX34 pad 2: /COL5 -> /COL6
- MX35 pad 2: /COL5 -> /COL6
- MX36 pad 2: /COL5 -> /COL7
- MX37 pad 2: /COL6 -> /COL7
- MX38 pad 2: /COL6 -> /COL7
- MX39 pad 2: /COL6 -> /COL7
- MX40 pad 2: /COL6 -> /COL7
- MX41 pad 2: /COL6 -> /COL8
- MX42 pad 2: /COL6 -> /COL8
- MX43 pad 2: /COL7 -> /COL8
- MX44 pad 2: /COL7 -> /COL8
- MX45 pad 2: /COL7 -> /COL8
- MX46 pad 2: /COL7 -> /COL9
- MX47 pad 2: /COL7 -> /COL9
- MX48 pad 2: /COL7 -> /COL9
- MX49 pad 2: /COL8 -> /COL9
- MX50 pad 2: /COL8 -> /COL9
- MX51 pad 2: /COL8 -> /COL10
- MX52 pad 2: /COL8 -> /COL10
- MX53 pad 2: /COL8 -> /COL10
- MX54 pad 2: /COL8 -> /COL10
- MX55 pad 2: /COL9 -> /COL10
- MX56 pad 2: /COL9 -> /COL11
- MX57 pad 2: /COL9 -> /COL11
- MX58 pad 2: /COL9 -> /COL11
- MX59 pad 2: /COL9 -> /COL11
- MX6 pad 2: /COL0 -> /COL1
- MX60 pad 2: /COL9 -> /COL11
- MX61 pad 1: Net-(D63-A) -> Net-(D61-A)
- MX61 pad 2: /COL10 -> /COL12
- MX62 pad 1: Net-(D64-A) -> Net-(D62-A)
- MX62 pad 2: /COL10 -> /COL12
- MX63 pad 1: Net-(D65-A) -> Net-(D63-A)
- MX63 pad 2: /COL10 -> /COL12
- MX64 pad 1: Net-(D66-A) -> Net-(D64-A)
- MX64 pad 2: /COL10 -> /COL12
- MX65 pad 1: Net-(D67-A) -> Net-(D65-A)
- MX65 pad 2: /COL10 -> /COL12
- MX66 pad 1: Net-(D68-A) -> Net-(D66-A)
- MX66 pad 2: /COL10 -> /COL13
- MX67 pad 1: Net-(D69-A) -> Net-(D67-A)
- MX67 pad 2: /COL11 -> /COL13
- MX68 pad 1: Net-(D70-A) -> Net-(D68-A)
- MX68 pad 2: /COL11 -> /COL13
- MX69 pad 1: Net-(D71-A) -> Net-(D69-A)
- MX69 pad 2: /COL11 -> /COL13
- MX70 pad 1: Net-(D72-A) -> Net-(D70-A)
- MX70 pad 2: /COL11 -> /COL13
- MX71 pad 1: Net-(D73-A) -> Net-(D71-A)
- MX71 pad 2: /COL11 -> /COL14
- MX72 pad 1: Net-(D74-A) -> Net-(D72-A)
- MX72 pad 2: /COL11 -> /COL14
- MX73 pad 1: Net-(D75-A) -> Net-(D73-A)
- MX73 pad 2: /COL12 -> /COL14
- MX74 pad 1: Net-(D76-A) -> Net-(D74-A)
- MX74 pad 2: /COL12 -> /COL14
- MX75 pad 1: Net-(D77-A) -> Net-(D75-A)
- MX75 pad 2: /COL12 -> /COL14
- MX76 pad 1: Net-(D78-A) -> Net-(D76-A)
- MX76 pad 2: /COL12 -> /COL15
- MX77 pad 1: Net-(D79-A) -> Net-(D77-A)
- MX77 pad 2: /COL12 -> /COL15
- MX78 pad 1: Net-(D80-A) -> Net-(D78-A)
- MX78 pad 2: /COL12 -> /COL15
- MX79 pad 1: Net-(D81-A) -> Net-(D79-A)
- MX79 pad 2: /COL13 -> /COL15
- MX80 pad 1: Net-(D82-A) -> Net-(D80-A)
- MX80 pad 2: /COL13 -> /COL15
- R1 pad 1: Net-(D62-K) -> Net-(D82-K)
- R2 pad 1: Net-(D61-K) -> Net-(D81-K)
- R3 pad 1: Net-(D62-K) -> Net-(D82-K)
Routing:
- net /COL7: track 215.3 -> 0.00 mm
- net /COL1: track 104.3 -> 0.00 mm
- net /COL0: track 98.5 -> 0.00 mm
- net /COL4: track 96.9 -> 0.00 mm
- net /COL9: track 95.3 -> 0.00 mm
- net /COL3: track 95.3 -> 0.00 mm
- net /COL2: track 95.3 -> 0.00 mm
- net /COL6: track 87.7 -> 0.00 mm
- net /COL8: track 57.2 -> 0.00 mm
- net Net-(D82-K): vias 0 -> 1
- net Net-(D81-K): vias 0 -> 1
- net Net-(D76-A): vias 1 -> 0
- net Net-(D62-K): vias 1 -> 0
- net Net-(D61-K): vias 1 -> 0
- net GND: vias 17 -> 19
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
Commit message: layout traces
Parts:
- moved D47 37.8 mm to (180.5, 71.8), turned to 180 degrees
- moved D48 37.8 mm to (193.2, 107.3), turned to 0 degrees
- moved D67 37.8 mm to (180.5, 92.1), turned to 180 degrees
- moved D68 37.8 mm to (193.2, 127.6), turned to 0 degrees
- moved D57 37.8 mm to (180.5, 81.9), turned to 180 degrees
- moved D58 37.8 mm to (193.2, 117.5), turned to 0 degrees
- moved D77 37.8 mm to (180.5, 102.2), turned to 180 degrees
- moved D78 37.8 mm to (193.2, 137.8), turned to 0 degrees
- moved D42 36.4 mm to (183.1, 66.7), turned to 180 degrees
- moved D43 36.4 mm to (190.7, 102.2), turned to 0 degrees
- moved D52 36.4 mm to (183.1, 76.8), turned to 180 degrees
- moved D53 36.4 mm to (190.7, 112.4), turned to 0 degrees
- moved D62 36.4 mm to (183.1, 87.0), turned to 180 degrees
- moved D63 36.4 mm to (190.7, 122.6), turned to 0 degrees
- moved D72 36.4 mm to (183.1, 97.2), turned to 180 degrees
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Routing:
- net GND: track 0.00 -> 401.5 mm, vias 19 -> 17
- net /COL1: track 0.00 -> 345.5 mm, vias 0 -> 1
- net /COL2: track 0.00 -> 338.9 mm
- net /COL0: track 0.00 -> 336.6 mm
- net /COL3: track 0.00 -> 289.3 mm, vias 0 -> 1
- net /COL15: track 0.00 -> 276.7 mm
- net /COL4: track 0.00 -> 270.3 mm, vias 0 -> 1
- net /ROW0: track 0.00 -> 250.8 mm
- net /COL5: track 0.00 -> 250.1 mm
- net /ROW2: track 0.00 -> 247.4 mm
- net /COL14: track 0.00 -> 247.0 mm, vias 0 -> 2
- net Net-(D81-K): track 0.00 -> 245.8 mm, vias 1 -> 0
- net /COL12: track 0.00 -> 237.2 mm, vias 0 -> 1
- net /COL13: track 0.00 -> 234.6 mm, vias 0 -> 1
- net /COL6: track 0.00 -> 233.2 mm, vias 0 -> 3
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
Commit message: new layout
Parts:
- removed D25, D40, D65, D70, D76, D77, D78, D79, D80: 1N4148, Diode_THT:D_DO-35_SOD27_P7.62mm_Horizontal
- removed MX25, MX40, MX65, MX70, MX76, MX77, MX78, MX79, MX80: SW_Push, lumberjack:MX
- added H12: M2, lumberjack:MountingHole_M2, F.Cu at (353.6, 131.0)
- MX10, MX15, MX20, MX45, MX5, MX50, MX55, MX60: footprint lumberjack:MX -> Button_Switch_Keyboard:SW_Cherry_MX_1.25u_PCB
- MX2, MX67: footprint lumberjack:MX -> Button_Switch_Keyboard:SW_Cherry_MX_1.50u_PCB
- MX3, MX30, MX35: footprint lumberjack:MX -> Button_Switch_Keyboard:SW_Cherry_MX_1.75u_PCB
- MX4, MX63: footprint lumberjack:MX -> Button_Switch_Keyboard:SW_Cherry_MX_2.25u_PCB
- MX59: footprint lumberjack:MX -> Button_Switch_Keyboard:SW_Cherry_MX_2.75u_PCB
- MX71: footprint lumberjack:MX -> Button_Switch_Keyboard:SW_Cherry_MX_2.00u_PCB
- moved MX35 151.4 mm to (224.9, 135.5)
- moved MX36 141.6 mm to (234.3, 64.3)
- moved MX37 141.6 mm to (234.3, 83.4)
- moved MX38 141.6 mm to (234.3, 102.4)
- moved MX39 141.6 mm to (234.3, 121.5)
- moved MX31 141.5 mm to (215.2, 64.3)
- moved MX32 141.5 mm to (215.2, 83.4)
- moved MX33 141.5 mm to (215.2, 102.4)
- moved MX34 141.5 mm to (215.2, 121.5)
- moved J4 110.7 mm to (-23.5, 69.9)
- moved J3 102.4 mm to (-30.2, 67.6)
- moved D38 89.8 mm to (199.8, 110.5), turned to 180 degrees
- moved D31 88.5 mm to (199.8, 68.0)
- moved D36 83.7 mm to (196.8, 72.2)
- moved D32 83.4 mm to (184.8, 68.0)
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Connections:
- D10 pad 1: /ROW4 -> /ROW3
- D15 pad 1: /ROW4 -> /ROW3
- D20 pad 1: /ROW4 -> /ROW3
- D30 pad 1: /ROW4 -> /ROW3
- D35 pad 1: /ROW4 -> /ROW3
- D45 pad 1: /ROW4 -> /ROW3
- D5 pad 1: /ROW4 -> /ROW3
- D50 pad 1: /ROW4 -> /ROW3
- D55 pad 1: /ROW4 -> /ROW3
- D60 pad 1: /ROW4 -> /ROW3
- D75 pad 1: /ROW4 -> /ROW3
- U2 pad 3: /ROW4 -> /ROW3
Routing:
- net GND: track 401.5 -> 0.00 mm, vias 17 -> 0
- net /COL1: track 345.5 -> 0.00 mm, vias 1 -> 0
- net /COL2: track 338.9 -> 0.00 mm
- net /COL0: track 336.6 -> 0.00 mm
- net /COL3: track 289.3 -> 0.00 mm, vias 1 -> 0
- net /COL15: track 276.7 -> 0.00 mm
- net /COL4: track 270.3 -> 0.00 mm, vias 1 -> 0
- net /ROW0: track 250.8 -> 0.00 mm
- net /COL5: track 250.1 -> 0.00 mm, vias 1 -> 0
- net /ROW2: track 247.4 -> 0.00 mm
- net /COL14: track 247.0 -> 0.00 mm, vias 2 -> 0
- net Net-(D81-K): track 245.8 -> 0.00 mm
- net /COL12: track 237.2 -> 0.00 mm, vias 1 -> 0
- net /COL13: track 234.6 -> 0.00 mm, vias 1 -> 0
- net /COL6: track 233.2 -> 0.00 mm, vias 3 -> 0
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Other:
- board size 404.3 x 94.2 mm -> 434.5 x 94.3 mm
