File: lumberjack.kicad_pcb (KiCad board)
At the start: 2 copper layers, 434.5 x 94.3 mm, 180 parts, among them J1 USB, J2 AVR_ISP_6, J3 JST, J4 JST, SW1 RESET, SW2 BOOT, U2 ATmega32A-P, Y1 16MHz

Commit message: middle part layout and traces
Parts:
- moved R6 105.2 mm to (88.1, 73.7), turned to 180 degrees
- moved J3 95.9 mm to (65.5, 73.7)
- moved J4 94.7 mm to (71.0, 76.0)
- moved J1 88.0 mm to (59.0, 60.9)
- moved R5 85.8 mm to (49.5, 73.7), turned to 0 degrees
- moved R1 75.9 mm to (141.0, 146.1), turned to 0 degrees
- moved C5 66.4 mm to (143.6, 127.0), turned to 0 degrees
- moved C3 63.6 mm to (138.4, 125.7)
- moved C4 62.6 mm to (143.5, 124.0), turned to 0 degrees
- moved R2 58.9 mm to (141.0, 142.2), turned to 0 degrees
- moved R3 53.7 mm to (163.8, 142.2), turned to 180 degrees
- moved R4 41.5 mm to (156.2, 146.1), turned to 0 degrees
- moved D2 21.4 mm to (129.6, 89.2)
- moved D27 21.4 mm to (126.8, 68.0)
- moved D1 21.1 mm to (113.6, 88.9)
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Connections:
- U2 pad 1: /COL0 -> /COL1
- U2 pad 14: /COL6 -> unconnected-(U2-PD0-Pad14)
- U2 pad 2: unconnected-(U2-PB1-Pad2) -> /COL0
- U2 pad 21: /COL1 -> /ROW1
- U2 pad 23: /COL7 -> /COL8
- U2 pad 24: /COL8 -> /COL7
- U2 pad 26: /LED2 -> /COL6
- U2 pad 27: /LED1 -> unconnected-(U2-PC5-Pad27)
- U2 pad 39: unconnected-(U2-PA1-Pad39) -> /LED1
- U2 pad 40: unconnected-(U2-PA0-Pad40) -> /LED2
- U2 pad 6: /ROW1 -> unconnected-(U2-PB5-Pad6)
Routing:
- net /COL14: track 0.00 -> 331.5 mm
- net /COL12: track 0.00 -> 322.2 mm
- net /COL13: track 0.00 -> 305.8 mm
- net /COL0: track 0.00 -> 266.4 mm
- net /COL11: track 0.00 -> 257.0 mm
- net Net-(D74-A): track 0.00 -> 239.1 mm
- net Net-(D75-A): track 0.00 -> 238.1 mm
- net /COL1: track 0.00 -> 237.6 mm
- net /COL10: track 0.00 -> 230.0 mm
- net /ROW3: track 0.00 -> 225.9 mm
- net GND: track 0.00 -> 224.6 mm
- net Net-(D60-A): track 0.00 -> 218.3 mm
- net Net-(D72-A): track 0.00 -> 218.2 mm
- net Net-(D71-A): track 0.00 -> 217.3 mm
- net /COL2: track 0.00 -> 216.1 mm
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
Commit message: usb mini and traces
Parts:
- removed J3: JST, Connector_JST:JST_SH_SM04B-SRSS-TB_1x04-1MP_P1.00mm_Horizontal
- removed J4: JST, lumberjack:S4B-ZRLFSN
- removed R5, R6: 5.1k, Resistor_THT:R_Axial_DIN0204_L3.6mm_D1.6mm_P7.62mm_Horizontal
- J1: value USB -> USB_B_Mini; footprint Connector_USB:USB_C_Receptacle_GCT_USB4085 -> lumberjack:USB_Mini-B; moved to F.Cu
- moved J1 82.2 mm to (-23.2, 64.0)
Connections:
- F1 pad 1: Net-(J3-Pin_1) -> Net-(J1-VBUS)
Routing:
- net Net-(D82-K): track 60.8 -> 286.0 mm
- net Net-(J1-VBUS): track 0.00 -> 223.2 mm
- net Net-(D81-K): track 28.6 -> 246.4 mm
- net GND: track 224.6 -> 23.1 mm
- net +5V: track 144.2 -> 192.7 mm, vias 0 -> 1
- net Net-(D27-A): track 91.7 -> 51.0 mm
- net Net-(J1-CC2): track 27.7 -> 0.00 mm
- net /COL4: track 63.5 -> 38.1 mm
- net Net-(J3-Pin_1): track 19.2 -> 0.00 mm
- net Net-(J1-CC1): track 14.2 -> 0.00 mm
- net Net-(D45-A): track 146.9 -> 144.0 mm
- net /COL2: track 216.1 -> 213.3 mm
- net Net-(D5-A): track 125.1 -> 124.2 mm
- net Net-(D10-A): track 102.6 -> 101.8 mm
- net Net-(D35-A): track 115.9 -> 116.8 mm
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
Commit message: gerber output
Parts:
- removed H5, H6: M2, lumberjack:MountingSlot_M2
- added H10: M2, lumberjack:MountingHole_M2, F.Cu at (320.0, 73.8)
- added H8: M2, lumberjack:MountingHole_M2, F.Cu at (4.70, 130.8)
- added H8: M2, lumberjack:MountingHole_M2, F.Cu at (4.70, 73.5)
- moved H10 76.1 mm to (243.8, 73.8)
- moved H8 38.0 mm to (42.7, 73.7)
Routing:
- net /COL4: track 38.1 -> 151.2 mm
- net /ROW1: track 127.7 -> 192.5 mm
- net +5V: track 192.7 -> 141.5 mm, vias 1 -> 0
- net /COL12: track 322.2 -> 281.1 mm, vias 0 -> 1
- net /ROW3: track 225.9 -> 237.9 mm
- net Net-(D55-A): track 191.5 -> 198.6 mm
- net Net-(D82-K): track 286.0 -> 291.5 mm
- net /ROW2: track 206.4 -> 211.9 mm
- net /COL13: track 305.8 -> 310.5 mm
- net /COL14: track 331.5 -> 336.2 mm
- net /COL10: track 230.0 -> 234.7 mm
- net /COL11: track 257.0 -> 261.7 mm
- net Net-(D35-A): track 116.8 -> 120.8 mm
- net Net-(D60-A): track 218.3 -> 215.0 mm
- net Net-(D44-A): track 93.9 -> 91.5 mm
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Other:
- board size 434.5 x 94.3 mm -> 434.9 x 94.2 mm
- board text removed: "POST"

Commit message: change dimensions to fit handrest
Parts:
- removed D1, D10, D11, D12, D13, D14, D15, D16, D17, D18, D19, D2, D20, D21, D22, D23, D24, D26, D27, D28, D29, D3, D30, D31, D32, D33, D34, D35, D36, D37, D38, D39, D4, D41, D42, D43, D44, D45, D46, D47, D48, D49, D5, D50, D51, D52, D53, D54, D55, D56, D57, D58, D59, D6, D60, D61, D62, D63, D64, D66, D67, D68, D69, D7, D71, D72, D73, D74, D75, D8, D9: 1N4148, Diode_THT:D_DO-35_SOD27_P7.62mm_Horizontal
- removed H7: M2, lumberjack:MountingSlot_M2
- removed J2: AVR_ISP_6, Connector_PinHeader_2.54mm:PinHeader_2x03_P2.54mm_Vertical
- removed MX1, MX11, MX12, MX13, MX14, MX16, MX17, MX18, MX19, MX21, MX22, MX23, MX24, MX26, MX27, MX28, MX29, MX31, MX32, MX33, MX34, MX36, MX37, MX38, MX39, MX41, MX42, MX43, MX44, MX46, MX47, MX48, MX49, MX51, MX52, MX53, MX54, MX56, MX57, MX58, MX6, MX61, MX62, MX64, MX66, MX68, MX69, MX72, MX73, MX74, MX75, MX8, MX9: SW_Push, lumberjack:MX
- removed MX10, MX15, MX20, MX45, MX5, MX50, MX55, MX60: SW_Push, Button_Switch_Keyboard:SW_Cherry_MX_1.25u_PCB
- removed MX2, MX67: SW_Push, Button_Switch_Keyboard:SW_Cherry_MX_1.50u_PCB
- removed MX3, MX30, MX35: SW_Push, Button_Switch_Keyboard:SW_Cherry_MX_1.75u_PCB
- removed MX4, MX63: SW_Push, Button_Switch_Keyboard:SW_Cherry_MX_2.25u_PCB
- removed MX59: SW_Push, Button_Switch_Keyboard:SW_Cherry_MX_2.75u_PCB
- removed MX7: SW_Push, lumberjack:MX_NTHSTH
- removed MX71: SW_Push, Button_Switch_Keyboard:SW_Cherry_MX_2.00u_PCB
- added D_1: 1N4148, Diode_THT:D_DO-35_SOD27_P7.62mm_Horizontal, F.Cu at (118.3, 207.2)
- added D_10: 1N4148, Diode_THT:D_DO-35_SOD27_P7.62mm_Horizontal, F.Cu at (118.3, 271.1)
- added D_11: 1N4148, Diode_THT:D_DO-35_SOD27_P7.62mm_Horizontal, F.Cu at (118.3, 200.8)
- added D_12: 1N4148, Diode_THT:D_DO-35_SOD27_P7.62mm_Horizontal, F.Cu at (118.3, 220.0)
- added D_13: 1N4148, Diode_THT:D_DO-35_SOD27_P7.62mm_Horizontal, F.Cu at (118.3, 236.0)
- added D_14: 1N4148, Diode_THT:D_DO-35_SOD27_P7.62mm_Horizontal, F.Cu at (118.3, 258.3)
- added D_15: 1N4148, Diode_THT:D_DO-35_SOD27_P7.62mm_Horizontal, F.Cu at (118.3, 274.3)
- added D_16: 1N4148, Diode_THT:D_DO-35_SOD27_P7.62mm_Horizontal, F.Cu at (118.3, 197.6)
- added D_17: 1N4148, Diode_THT:D_DO-35_SOD27_P7.62mm_Horizontal, F.Cu at (118.3, 216.8)
- added D_18: 1N4148, Diode_THT:D_DO-35_SOD27_P7.62mm_Horizontal, F.Cu at (118.3, 239.2)
- added D_19: 1N4148, Diode_THT:D_DO-35_SOD27_P7.62mm_Horizontal, F.Cu at (118.3, 255.1)
- added D_2: 1N4148, Diode_THT:D_DO-35_SOD27_P7.62mm_Horizontal, F.Cu at (118.3, 226.4)
- added D_20: 1N4148, Diode_THT:D_DO-35_SOD27_P7.62mm_Horizontal, F.Cu at (118.3, 277.5)
- added D_21: 1N4148, Diode_THT:D_DO-35_SOD27_P7.62mm_Horizontal, F.Cu at (118.3, 194.4)
- added D_22: 1N4148, Diode_THT:D_DO-35_SOD27_P7.62mm_Horizontal, F.Cu at (118.3, 213.6)
- added D_23: 1N4148, Diode_THT:D_DO-35_SOD27_P7.62mm_Horizontal, F.Cu at (118.3, 242.4)
- added D_24: 1N4148, Diode_THT:D_DO-35_SOD27_P7.62mm_Horizontal, F.Cu at (118.3, 252.0)
- added D_25: 1N4148, Diode_THT:D_DO-35_SOD27_P7.62mm_Horizontal, F.Cu at (118.3, 191.2)
- added D_26: 1N4148, Diode_THT:D_DO-35_SOD27_P7.62mm_Horizontal, F.Cu at (118.3, 210.4)
- added D_27: 1N4148, Diode_THT:D_DO-35_SOD27_P7.62mm_Horizontal, F.Cu at (118.3, 245.6)
- added D_28: 1N4148, Diode_THT:D_DO-35_SOD27_P7.62mm_Horizontal, F.Cu at (118.3, 248.8)
- added D_29: 1N4148, Diode_THT:D_DO-35_SOD27_P7.62mm_Horizontal, F.Cu at (118.3, 280.7)
- added D_3: 1N4148, Diode_THT:D_DO-35_SOD27_P7.62mm_Horizontal, F.Cu at (118.3, 229.6)
- added D_30: 1N4148, Diode_THT:D_DO-35_SOD27_P7.62mm_Horizontal, F.Cu at (150.6, 191.2)
- added D_31: 1N4148, Diode_THT:D_DO-35_SOD27_P7.62mm_Horizontal, F.Cu at (150.6, 220.0)
- added D_32: 1N4148, Diode_THT:D_DO-35_SOD27_P7.62mm_Horizontal, F.Cu at (150.6, 245.6)
- added D_33: 1N4148, Diode_THT:D_DO-35_SOD27_P7.62mm_Horizontal, F.Cu at (150.6, 280.7)
- added D_34: 1N4148, Diode_THT:D_DO-35_SOD27_P7.62mm_Horizontal, F.Cu at (147.1, 273.4)
- added D_35: 1N4148, Diode_THT:D_DO-35_SOD27_P7.62mm_Horizontal, F.Cu at (150.6, 194.4)
- added D_36: 1N4148, Diode_THT:D_DO-35_SOD27_P7.62mm_Horizontal, F.Cu at (150.6, 223.2)
- added D_37: 1N4148, Diode_THT:D_DO-35_SOD27_P7.62mm_Horizontal, F.Cu at (150.6, 248.8)
- added D_38: 1N4148, Diode_THT:D_DO-35_SOD27_P7.62mm_Horizontal, F.Cu at (150.6, 277.5)
- added D_39: 1N4148, Diode_THT:D_DO-35_SOD27_P7.62mm_Horizontal, F.Cu at (150.6, 197.6)
- added D_4: 1N4148, Diode_THT:D_DO-35_SOD27_P7.62mm_Horizontal, F.Cu at (118.3, 264.7)
- added D_40: 1N4148, Diode_THT:D_DO-35_SOD27_P7.62mm_Horizontal, F.Cu at (150.6, 226.4)
- added D_41: 1N4148, Diode_THT:D_DO-35_SOD27_P7.62mm_Horizontal, F.Cu at (150.6, 252.0)
- added D_42: 1N4148, Diode_THT:D_DO-35_SOD27_P7.62mm_Horizontal, F.Cu at (150.6, 274.3)
- added D_43: 1N4148, Diode_THT:D_DO-35_SOD27_P7.62mm_Horizontal, F.Cu at (143.6, 273.4)
- added D_44: 1N4148, Diode_THT:D_DO-35_SOD27_P7.62mm_Horizontal, F.Cu at (150.6, 200.8)
- added D_45: 1N4148, Diode_THT:D_DO-35_SOD27_P7.62mm_Horizontal, F.Cu at (150.6, 229.6)
- added D_46: 1N4148, Diode_THT:D_DO-35_SOD27_P7.62mm_Horizontal, F.Cu at (150.6, 255.1)
- added D_47: 1N4148, Diode_THT:D_DO-35_SOD27_P7.62mm_Horizontal, F.Cu at (150.6, 271.1)
- added D_48: 1N4148, Diode_THT:D_DO-35_SOD27_P7.62mm_Horizontal, F.Cu at (140.0, 273.4)
- added D_49: 1N4148, Diode_THT:D_DO-35_SOD27_P7.62mm_Horizontal, F.Cu at (150.6, 204.0)
- added D_5: 1N4148, Diode_THT:D_DO-35_SOD27_P7.62mm_Horizontal, F.Cu at (118.3, 267.9)
- added D_50: 1N4148, Diode_THT:D_DO-35_SOD27_P7.62mm_Horizontal, F.Cu at (150.6, 232.8)
- added D_51: 1N4148, Diode_THT:D_DO-35_SOD27_P7.62mm_Horizontal, F.Cu at (150.6, 258.3)
- added D_52: 1N4148, Diode_THT:D_DO-35_SOD27_P7.62mm_Horizontal, F.Cu at (150.6, 267.9)
- added D_53: 1N4148, Diode_THT:D_DO-35_SOD27_P7.62mm_Horizontal, F.Cu at (136.5, 273.4)
- added D_54: 1N4148, Diode_THT:D_DO-35_SOD27_P7.62mm_Horizontal, F.Cu at (150.6, 207.2)
- added D_55: 1N4148, Diode_THT:D_DO-35_SOD27_P7.62mm_Horizontal, F.Cu at (150.6, 236.0)
- added D_56: 1N4148, Diode_THT:D_DO-35_SOD27_P7.62mm_Horizontal, F.Cu at (150.6, 261.5)
- added D_57: 1N4148, Diode_THT:D_DO-35_SOD27_P7.62mm_Horizontal, F.Cu at (122.3, 273.4)
- added D_58: 1N4148, Diode_THT:D_DO-35_SOD27_P7.62mm_Horizontal, F.Cu at (132.9, 273.4)
- added D_59: 1N4148, Diode_THT:D_DO-35_SOD27_P7.62mm_Horizontal, F.Cu at (150.6, 210.4)
- added D_6: 1N4148, Diode_THT:D_DO-35_SOD27_P7.62mm_Horizontal, F.Cu at (118.3, 204.0)
- added D_60: 1N4148, Diode_THT:D_DO-35_SOD27_P7.62mm_Horizontal, F.Cu at (150.6, 239.2)
- added D_61: 1N4148, Diode_THT:D_DO-35_SOD27_P7.62mm_Horizontal, F.Cu at (150.6, 264.7)
- added D_62: 1N4148, Diode_THT:D_DO-35_SOD27_P7.62mm_Horizontal, F.Cu at (129.4, 273.4)
- added D_63: 1N4148, Diode_THT:D_DO-35_SOD27_P7.62mm_Horizontal, F.Cu at (150.6, 213.6)
- added D_64: 1N4148, Diode_THT:D_DO-35_SOD27_P7.62mm_Horizontal, F.Cu at (150.6, 242.4)
- added D_65: 1N4148, Diode_THT:D_DO-35_SOD27_P7.62mm_Horizontal, F.Cu at (125.8, 273.4)
- added D_66: 1N4148, Diode_THT:D_DO-35_SOD27_P7.62mm_Horizontal, F.Cu at (150.6, 216.8)
- added D_7: 1N4148, Diode_THT:D_DO-35_SOD27_P7.62mm_Horizontal, F.Cu at (118.3, 223.2)
- added D_8: 1N4148, Diode_THT:D_DO-35_SOD27_P7.62mm_Horizontal, F.Cu at (118.3, 232.8)
- added D_9: 1N4148, Diode_THT:D_DO-35_SOD27_P7.62mm_Horizontal, F.Cu at (118.3, 261.5)
- added K_1: KEYSW, Button_Switch_Keyboard:SW_Cherry_MX_1.00u_PCB, F.Cu at (6.45, 193.2)
- added K_10: KEYSW, Button_Switch_Keyboard:SW_Cherry_MX_1.25u_PCB, F.Cu at (18.5, 269.6)
- added K_11: KEYSW, Button_Switch_Keyboard:SW_Cherry_MX_1.00u_PCB, F.Cu at (44.6, 193.2)
- added K_12: KEYSW, Button_Switch_Keyboard:SW_Cherry_MX_1.00u_PCB, F.Cu at (44.6, 212.3)
- added K_13: KEYSW, Button_Switch_Keyboard:SW_Cherry_MX_1.00u_PCB, F.Cu at (44.6, 231.4)
- added K_14: KEYSW, Button_Switch_Keyboard:SW_Cherry_MX_1.00u_PCB, F.Cu at (44.6, 250.5)
- added K_15: KEYSW, Button_Switch_Keyboard:SW_Cherry_MX_1.25u_PCB, F.Cu at (42.4, 269.7)
- added K_16: KEYSW, Button_Switch_Keyboard:SW_Cherry_MX_1.00u_PCB, F.Cu at (63.7, 193.2)
- added K_17: KEYSW, Button_Switch_Keyboard:SW_Cherry_MX_1.00u_PCB, F.Cu at (63.7, 212.3)
- added K_18: KEYSW, Button_Switch_Keyboard:SW_Cherry_MX_1.00u_PCB, F.Cu at (63.7, 231.4)
- added K_19: KEYSW, Button_Switch_Keyboard:SW_Cherry_MX_1.00u_PCB, F.Cu at (63.7, 250.5)
- added K_2: KEYSW, Button_Switch_Keyboard:SW_Cherry_MX_1.50u_PCB, F.Cu at (1.68, 212.3)
- added K_20: KEYSW, Button_Switch_Keyboard:SW_Cherry_MX_1.25u_PCB, F.Cu at (66.2, 269.6)
- added K_21: KEYSW, Button_Switch_Keyboard:SW_Cherry_MX_1.00u_PCB, F.Cu at (82.8, 193.2)
- added K_22: KEYSW, Button_Switch_Keyboard:SW_Cherry_MX_1.00u_PCB, F.Cu at (82.8, 212.3)
- added K_23: KEYSW, Button_Switch_Keyboard:SW_Cherry_MX_1.00u_PCB, F.Cu at (82.8, 231.4)
- added K_24: KEYSW, Button_Switch_Keyboard:SW_Cherry_MX_1.00u_PCB, F.Cu at (82.8, 250.5)
- added K_25: KEYSW, Button_Switch_Keyboard:SW_Cherry_MX_1.00u_PCB, F.Cu at (101.9, 193.2)
- added K_26: KEYSW, Button_Switch_Keyboard:SW_Cherry_MX_1.00u_PCB, F.Cu at (101.9, 212.3)
- added K_27: KEYSW, Button_Switch_Keyboard:SW_Cherry_MX_1.00u_PCB, F.Cu at (101.9, 231.4)
- added K_28: KEYSW, Button_Switch_Keyboard:SW_Cherry_MX_1.00u_PCB, F.Cu at (101.9, 250.5)
- added K_29: KEYSW, Button_Switch_Keyboard:SW_Cherry_MX_1.75u_PCB, F.Cu at (94.8, 269.6)
- added K_3: KEYSW, Button_Switch_Keyboard:SW_Cherry_MX_1.75u_PCB, F.Cu at (-0.70, 231.4)
- added K_30: KEYSW, Button_Switch_Keyboard:SW_Cherry_MX_1.00u_PCB, F.Cu at (173.9, 193.2)
- added K_31: KEYSW, Button_Switch_Keyboard:SW_Cherry_MX_1.00u_PCB, F.Cu at (173.9, 212.3)
- added K_32: KEYSW, Button_Switch_Keyboard:SW_Cherry_MX_1.00u_PCB, F.Cu at (173.9, 231.4)
- added K_33: KEYSW, Button_Switch_Keyboard:SW_Cherry_MX_1.00u_PCB, F.Cu at (173.9, 250.5)
- added K_34: KEYSW, Button_Switch_Keyboard:SW_Cherry_MX_1.75u_PCB, F.Cu at (181.1, 269.6)
- added K_35: KEYSW, Button_Switch_Keyboard:SW_Cherry_MX_1.00u_PCB, F.Cu at (193.0, 193.2)
- added K_36: KEYSW, Button_Switch_Keyboard:SW_Cherry_MX_1.00u_PCB, F.Cu at (193.0, 212.3)
- added K_37: KEYSW, Button_Switch_Keyboard:SW_Cherry_MX_1.00u_PCB, F.Cu at (193.0, 231.4)
- added K_38: KEYSW, Button_Switch_Keyboard:SW_Cherry_MX_1.00u_PCB, F.Cu at (193.0, 250.5)
- added K_39: KEYSW, Button_Switch_Keyboard:SW_Cherry_MX_1.00u_PCB, F.Cu at (212.1, 193.2)
- added K_4: KEYSW, Button_Switch_Keyboard:SW_Cherry_MX_2.25u_PCB, F.Cu at (-5.46, 250.5)
- added K_40: KEYSW, Button_Switch_Keyboard:SW_Cherry_MX_1.00u_PCB, F.Cu at (212.1, 212.3)
- added K_41: KEYSW, Button_Switch_Keyboard:SW_Cherry_MX_1.00u_PCB, F.Cu at (212.1, 231.4)
- added K_42: KEYSW, Button_Switch_Keyboard:SW_Cherry_MX_1.00u_PCB, F.Cu at (212.1, 250.5)
- added K_43: KEYSW, Button_Switch_Keyboard:SW_Cherry_MX_1.25u_PCB, F.Cu at (209.8, 269.6)
- added K_44: KEYSW, Button_Switch_Keyboard:SW_Cherry_MX_1.00u_PCB, F.Cu at (231.2, 193.2)
- added K_45: KEYSW, Button_Switch_Keyboard:SW_Cherry_MX_1.00u_PCB, F.Cu at (231.2, 212.3)
- added K_46: KEYSW, Button_Switch_Keyboard:SW_Cherry_MX_1.00u_PCB, F.Cu at (231.2, 231.4)
- added K_47: KEYSW, Button_Switch_Keyboard:SW_Cherry_MX_1.00u_PCB, F.Cu at (231.2, 250.5)
- added K_48: KEYSW, Button_Switch_Keyboard:SW_Cherry_MX_1.25u_PCB, F.Cu at (233.7, 269.6)
- added K_49: KEYSW, Button_Switch_Keyboard:SW_Cherry_MX_1.00u_PCB, F.Cu at (250.3, 193.2)
- added K_5: KEYSW, Button_Switch_Keyboard:SW_Cherry_MX_1.25u_PCB, F.Cu at (-5.24, 269.6)
- added K_50: KEYSW, Button_Switch_Keyboard:SW_Cherry_MX_1.00u_PCB, F.Cu at (250.3, 212.3)
- added K_51: KEYSW, Button_Switch_Keyboard:SW_Cherry_MX_1.00u_PCB, F.Cu at (250.3, 231.4)
- added K_52: KEYSW, Button_Switch_Keyboard:SW_Cherry_MX_1.00u_PCB, F.Cu at (250.3, 250.5)
- added K_53: KEYSW, Button_Switch_Keyboard:SW_Cherry_MX_1.00u_PCB, F.Cu at (255.1, 269.6)
- added K_54: KEYSW, Button_Switch_Keyboard:SW_Cherry_MX_1.00u_PCB, F.Cu at (269.4, 193.2)
- added K_55: KEYSW, Button_Switch_Keyboard:SW_Cherry_MX_1.00u_PCB, F.Cu at (269.4, 212.3)
- added K_56: KEYSW, Button_Switch_Keyboard:SW_Cherry_MX_1.00u_PCB, F.Cu at (269.4, 231.4)
- added K_57: KEYSW, Button_Switch_Keyboard:SW_Cherry_MX_2.75u_PCB, F.Cu at (286.1, 250.5)
- added K_58: KEYSW, Button_Switch_Keyboard:SW_Cherry_MX_1.00u_PCB, F.Cu at (274.2, 269.6)
- added K_59: KEYSW, Button_Switch_Keyboard:SW_Cherry_MX_1.00u_PCB, F.Cu at (288.5, 193.2)
- added K_6: KEYSW, Button_Switch_Keyboard:SW_Cherry_MX_1.00u_PCB, F.Cu at (25.5, 193.2)
- added K_60: KEYSW, Button_Switch_Keyboard:SW_Cherry_MX_1.00u_PCB, F.Cu at (288.5, 212.3)
- added K_61: KEYSW, Button_Switch_Keyboard:SW_Cherry_MX_2.25u_PCB, F.Cu at (300.4, 231.4)
- added K_62: KEYSW, Button_Switch_Keyboard:SW_Cherry_MX_1.00u_PCB, F.Cu at (293.3, 269.6)
- added K_63: KEYSW, Button_Switch_Keyboard:SW_Cherry_MX_1.00u_PCB, F.Cu at (307.6, 193.2)
- added K_64: KEYSW, Button_Switch_Keyboard:SW_Cherry_MX_1.50u_PCB, F.Cu at (312.4, 212.3)
- added K_65: KEYSW, Button_Switch_Keyboard:SW_Cherry_MX_1.00u_PCB, F.Cu at (312.4, 269.6)
- added K_66: KEYSW, Button_Switch_Keyboard:SW_Cherry_MX_1.00u_PCB, F.Cu at (326.7, 193.2)
- added K_7: KEYSW, Button_Switch_Keyboard:SW_Cherry_MX_1.00u_PCB, F.Cu at (25.6, 212.3)
- added K_8: KEYSW, Button_Switch_Keyboard:SW_Cherry_MX_1.00u_PCB, F.Cu at (25.6, 231.4)
- added K_9: KEYSW, Button_Switch_Keyboard:SW_Cherry_MX_1.00u_PCB, F.Cu at (25.6, 250.5)
- moved H2 223.0 mm to (89.8, 265.1)
- moved SW1 192.2 mm to (132.7, 267.5), turned to 180 degrees
- moved F1 182.6 mm to (-20.0, 210.8), turned to 180 degrees
- moved D82 181.3 mm to (-26.4, 203.2)
- moved D81 169.5 mm to (-15.4, 203.2)
- moved SW2 160.1 mm to (142.7, 267.5), turned to 180 degrees
- moved H11 157.2 mm to (181.1, 265.1)
- moved H1 153.3 mm to (89.8, 207.8)
- moved H10 148.0 mm to (180.8, 207.8)
- moved H8 144.6 mm to (-11.7, 217.2)
- moved H10 143.0 mm to (321.1, 216.8)
- moved R7 142.4 mm to (124.4, 198.4), turned to 90 degrees
- moved U2 141.2 mm to (130.8, 209.1)
- moved Y1 138.7 mm to (124.4, 227.2), turned to 90 degrees
- moved H4 135.5 mm to (238.3, 265.1)
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Connections:
- SW2 pad 1: /COL3 -> COL3
- U2 pad 1: /COL1 -> COL0
- U2 pad 15: /COL5 -> unconnected-(U2-PD1-Pad15)
- U2 pad 18: /COL4 -> ROW2
- U2 pad 19: /COL3 -> ROW3
- U2 pad 2: /COL0 -> COL1
- U2 pad 20: /COL2 -> ROW4
- U2 pad 21: /ROW1 -> /COL15
- U2 pad 22: /ROW0 -> COL14
- U2 pad 23: /COL8 -> COL13
- U2 pad 24: /COL7 -> COL12
- U2 pad 25: /COL9 -> COL11
- U2 pad 26: /COL6 -> COL10
- U2 pad 27: unconnected-(U2-PC5-Pad27) -> COL9
- U2 pad 28: unconnected-(U2-PC6-Pad28) -> COL8
- U2 pad 29: unconnected-(U2-PC7-Pad29) -> COL7
- U2 pad 3: /ROW3 -> COL2
- U2 pad 33: /COL10 -> COL6
- U2 pad 34: /COL11 -> unconnected-(U2-PA6-Pad34)
- U2 pad 35: /COL12 -> unconnected-(U2-PA5-Pad35)
- U2 pad 36: /COL13 -> unconnected-(U2-PA4-Pad36)
- U2 pad 37: /COL14 -> ROW0
- U2 pad 38: /COL15 -> ROW1
- U2 pad 39: /LED1 -> /LED2
- U2 pad 4: /ROW3 -> COL3
- U2 pad 40: /LED2 -> /LED1
- U2 pad 5: /ROW2 -> COL4
- U2 pad 6: unconnected-(U2-PB5-Pad6) -> COL5
Routing:
- net /COL14: track 336.2 -> 0.00 mm
- net /COL13: track 310.5 -> 0.00 mm
- net COL13: track 0.00 -> 298.8 mm
- net COL12: track 0.00 -> 282.1 mm
- net /COL12: track 281.1 -> 0.00 mm, vias 1 -> 0
- net /COL0: track 265.5 -> 0.00 mm
- net /COL11: track 261.7 -> 0.00 mm
- net COL11: track 0.00 -> 251.3 mm
- net COL14: track 0.00 -> 246.4 mm
- net COL3: track 0.00 -> 243.2 mm
- net COL0: track 0.00 -> 241.8 mm
- net Net-(D74-A): track 239.0 -> 0.00 mm
- net Net-(D75-A): track 238.0 -> 0.00 mm
- net /ROW3: track 237.9 -> 0.00 mm
- net /COL1: track 237.3 -> 0.00 mm
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Other:
- board size 434.9 x 94.2 mm -> 363.2 x 95.5 mm
- board text removed: "GND"
- board text removed: "ISP"
- board text removed: "JLCJLCJLCJLC"
- board text removed: "MISO"
- board text removed: "MOSI"
- board text removed: "RST"
- board text removed: "SCLK"
- board text removed: "VCC"
- board text removed: "rev1.7 03/2023"

Commit message: replace mcu with teensy
Parts:
- removed C1, C2: 22p, Capacitor_THT:C_Disc_D3.0mm_W1.6mm_P2.50mm
- removed C3: 4.7u, Capacitor_THT:CP_Radial_D4.0mm_P1.50mm
- removed C4, C5: 100n, Capacitor_THT:C_Disc_D4.3mm_W1.9mm_P5.00mm
- removed D81, D82: 3.6V, Diode_THT:D_DO-35_SOD27_P7.62mm_Horizontal
- removed F1: 100mA, Fuse:Fuse_Bourns_MF-RHT100
- removed J1: USB_B_Mini, lumberjack:USB_Mini-B
- removed LED1: RED, LED_THT:LED_D3.0mm
- removed LED2: GREEN, LED_THT:LED_D3.0mm
- removed R1, R7, R8: 1.5k, Resistor_THT:R_Axial_DIN0204_L3.6mm_D1.6mm_P7.62mm_Horizontal
- removed R2, R3: 75R, Resistor_THT:R_Axial_DIN0204_L3.6mm_D1.6mm_P7.62mm_Horizontal
- removed R4: 10k, Resistor_THT:R_Axial_DIN0204_L3.6mm_D1.6mm_P7.62mm_Horizontal
- removed SW2: BOOT, Button_Switch_THT:SW_PUSH_6mm
- removed U2: ATmega32A-P, Package_DIP:DIP-40_W15.24mm
- removed Y1: 16MHz, Crystal:Crystal_HC49-4H_Vertical
- added D1: 1N4148, Diode_THT:D_DO-35_SOD27_P7.62mm_Horizontal, F.Cu at (134.1, 228.6)
- added U1: Teensy2.0_(C), lumberjack:Teensy2.0, F.Cu at (135.4, 204.5)
- SW1: value RESET -> RotaryEncoder_Switch; footprint Button_Switch_THT:SW_PUSH_6mm -> Potentiometer_THT:Potentiometer_Bourns_PTV09A-1_Single_Vertical
- moved D_52 46.1 mm to (144.2, 222.2), turned to 180 degrees
- moved D_28 30.8 mm to (115.6, 279.4), turned to 0 degrees
- moved D_3 27.1 mm to (115.6, 256.5), turned to 0 degrees
- moved D_5 24.7 mm to (134.0, 248.9)
- moved D_15 23.7 mm to (134.0, 256.5)
- moved SW1 23.7 mm to (137.2, 244.2), turned to 90 degrees
- moved D_24 23.7 mm to (119.4, 275.6)
- moved D_53 23.5 mm to (123.2, 292.7), turned to 0 degrees
- moved D_26 23.4 mm to (115.6, 233.7), turned to 0 degrees
- moved D_47 23.1 mm to (144.2, 248.9), turned to 180 degrees
- moved D_29 22.8 mm to (134.0, 264.2)
- moved D_10 21.9 mm to (130.2, 252.7), turned to 0 degrees
- moved D_20 20.9 mm to (130.2, 260.4), turned to 0 degrees
- moved D_8 20.0 mm to (119.4, 252.7)
- moved D_34 19.7 mm to (141.0, 292.1), turned to 180 degrees
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Connections:
- SW1 pad 1: Net-(U2-~{RESET}) -> ENC_A
- SW1 pad 2: GND -> unconnected-(SW1-Pad2)
Routing:
- net COL13: track 298.8 -> 0.00 mm
- net +5V: track 288.8 -> 0.00 mm
- net COL12: track 282.1 -> 0.00 mm
- net COL11: track 251.3 -> 0.00 mm
- net COL14: track 246.4 -> 0.00 mm
- net Net-(D82-K): track 232.3 -> 0.00 mm
- net COL10: track 209.8 -> 0.00 mm
- net Net-(D81-K): track 209.6 -> 0.00 mm
- net Net-(D_65-A): track 194.5 -> 0.00 mm
- net COL9: track 191.1 -> 0.00 mm
- net COL8: track 171.4 -> 0.00 mm
- net Net-(D_62-A): track 170.0 -> 0.00 mm
- net Net-(D_57-A): track 169.5 -> 0.00 mm
- net COL3: track 243.2 -> 77.4 mm
- net COL0: track 241.8 -> 81.4 mm
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- added copper zone on B.Cu, net unconnected-(SW1-Pad2)
- added copper zone on F.Cu, net unconnected-(SW1-Pad2)
- removed copper zone on B.Cu, net GND
- removed copper zone on F.Cu, net GND

Commit message: add cirque trackpad
Parts:
- removed D1: 1N4148, Diode_THT:D_DO-35_SOD27_P7.62mm_Horizontal
- removed the H10 at (180.8, 207.8)
- removed the H10 at (321.1, 216.8)
- removed H2: M2, lumberjack:MountingHole_M2
- removed the H8 at (51.4, 207.0)
- removed the H8 at (-23.6, 256.2)
- removed the H8 at (-11.7, 217.2)
- removed SW1: RotaryEncoder_Switch, Potentiometer_THT:Potentiometer_Bourns_PTV09A-1_Single_Vertical
- added D_67: 1N4148, Diode_THT:D_DO-35_SOD27_P7.62mm_Horizontal, B.Cu at (319.0, 118.1)
- added D_68: 1N4148, Diode_THT:D_DO-35_SOD27_P7.62mm_Horizontal, B.Cu at (319.2, 104.8)
- added H10: M2, lumberjack:MountingHole_M2, F.Cu at (66.7, 47.6)
- added H5: M2, lumberjack:MountingHole_M2, F.Cu at (-9.53, 38.1)
- added H6: M2, lumberjack:MountingHole_M2, F.Cu at (257.2, 104.8)
- added H8: M2, lumberjack:MountingHole_M2, F.Cu at (-9.53, 114.3)
- added K_67: KEYSW, Button_Switch_Keyboard:SW_Cherry_MX_1.00u_PCB, F.Cu at (312.1, 109.2)
- added K_68: KEYSW, Button_Switch_Keyboard:SW_Cherry_MX_1.00u_PCB, F.Cu at (331.2, 109.2)
- added U2: Cirque40mm, lumberjack:cirque_40mm, F.Cu at (152.0, 85.7)
- D_1, D_10, D_11, D_12, D_13, D_14, D_15, D_16, D_17, D_18, D_19, D_2, D_20, D_21, D_22, D_23, D_24, D_25, D_26, D_27, D_28, D_29, D_3, D_30, D_31, D_32, D_33, D_34, D_35, D_36, D_37, D_38, D_39, D_4, D_40, D_41, D_42, D_43, D_44, D_45, D_46, D_47, D_48, D_49, D_5, D_50, D_51, D_52, D_53, D_54, D_55, D_56, D_57, D_58, D_59, D_6, D_62, D_63, D_64, D_65, D_66, D_7, D_8, D_9: moved to B.Cu
- K_10, K_15, K_20, K_48, K_5: footprint Button_Switch_Keyboard:SW_Cherry_MX_1.25u_PCB -> Button_Switch_Keyboard:SW_Cherry_MX_1.00u_PCB
- K_16: footprint Button_Switch_Keyboard:SW_Cherry_MX_1.00u_PCB -> Button_Switch_Keyboard:SW_Cherry_MX_1.50u_PCB
- K_2: footprint Button_Switch_Keyboard:SW_Cherry_MX_1.50u_PCB -> Button_Switch_Keyboard:SW_Cherry_MX_1.00u_PCB
- K_29: footprint Button_Switch_Keyboard:SW_Cherry_MX_1.75u_PCB -> Button_Switch_Keyboard:SW_Cherry_MX_1.50u_PCB
- K_3, K_34: footprint Button_Switch_Keyboard:SW_Cherry_MX_1.75u_PCB -> Button_Switch_Keyboard:SW_Cherry_MX_1.00u_PCB
- K_30, K_59, K_62: footprint Button_Switch_Keyboard:SW_Cherry_MX_1.00u_PCB -> Button_Switch_Keyboard:SW_Cherry_MX_1.75u_PCB
- K_4, K_61: footprint Button_Switch_Keyboard:SW_Cherry_MX_2.25u_PCB -> Button_Switch_Keyboard:SW_Cherry_MX_1.00u_PCB
- K_42: footprint Button_Switch_Keyboard:SW_Cherry_MX_1.00u_PCB -> Button_Switch_Keyboard:SW_Cherry_MX_2.25u_PCB
- K_43: footprint Button_Switch_Keyboard:SW_Cherry_MX_1.25u_PCB -> Button_Switch_Keyboard:SW_Cherry_MX_2.25u_PCB
- K_54: footprint Button_Switch_Keyboard:SW_Cherry_MX_1.00u_PCB -> Button_Switch_Keyboard:SW_Cherry_MX_2.75u_PCB
- K_55, K_56, K_58, K_63: footprint Button_Switch_Keyboard:SW_Cherry_MX_1.00u_PCB -> Button_Switch_Keyboard:SW_Cherry_MX_1.25u_PCB
- K_57: footprint Button_Switch_Keyboard:SW_Cherry_MX_2.75u_PCB -> Button_Switch_Keyboard:SW_Cherry_MX_1.25u_PCB
- K_64: footprint Button_Switch_Keyboard:SW_Cherry_MX_1.50u_PCB -> Button_Switch_Keyboard:SW_Cherry_MX_1.25u_PCB
- moved K_15 384.5 mm to (345.4, 33.0)
- moved H9 357.7 mm to (342.9, 57.1)
- moved K_14 355.9 mm to (326.4, 33.0)
- moved K_10 331.1 mm to (250.2, 33.0)
- moved K_13 329.2 mm to (307.3, 33.0)
- moved K_29 321.3 mm to (331.2, 52.1)
- moved D_14 311.2 mm to (333.3, 41.9), turned to 90 degrees
- moved K_12 302.5 mm to (288.3, 33.0)
- moved K_9 299.3 mm to (231.1, 33.0)
- moved H12 295.5 mm to (66.7, 104.8)
- moved D_28 295.3 mm to (314.3, 61.0), turned to 90 degrees
- moved D_15 288.7 mm to (333.4, 47.8), turned to 0 degrees
- moved D_29 288.0 mm to (338.1, 61.0), turned to 90 degrees
- moved D_13 286.9 mm to (314.3, 41.9), turned to 90 degrees
- moved K_28 285.6 mm to (307.3, 52.1)
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Connections:
- D_10 pad 1: ROW4 -> ROW0
- D_12 pad 1: ROW1 -> ROW0
- D_13 pad 1: ROW2 -> ROW0
- D_14 pad 1: ROW3 -> ROW0
- D_15 pad 1: ROW4 -> ROW0
- D_16 pad 1: ROW0 -> ROW1
- D_18 pad 1: ROW2 -> ROW1
- D_19 pad 1: ROW3 -> ROW1
- D_2 pad 1: ROW1 -> ROW0
- D_20 pad 1: ROW4 -> ROW1
- D_21 pad 1: ROW0 -> ROW1
- D_23 pad 1: ROW2 -> ROW1
- D_24 pad 1: ROW3 -> ROW1
- D_25 pad 1: ROW0 -> ROW1
- D_27 pad 1: ROW2 -> ROW1
- D_28 pad 1: ROW3 -> ROW1
- D_29 pad 1: ROW4 -> ROW1
- D_3 pad 1: ROW2 -> ROW0
- D_30 pad 1: ROW0 -> ROW2
- D_31 pad 1: ROW1 -> ROW2
- D_33 pad 1: ROW3 -> ROW2
- D_34 pad 1: ROW4 -> ROW2
- D_35 pad 1: ROW0 -> ROW2
- D_36 pad 1: ROW1 -> ROW2
- D_38 pad 1: ROW3 -> ROW2
- D_39 pad 1: ROW0 -> ROW2
- D_4 pad 1: ROW3 -> ROW0
- D_40 pad 1: ROW1 -> ROW2
- D_42 pad 1: ROW3 -> ROW2
- D_43 pad 1: ROW4 -> ROW3
- D_44 pad 1: ROW0 -> ROW3
- D_45 pad 1: ROW1 -> ROW3
- D_46 pad 1: ROW2 -> ROW3
- D_48 pad 1: ROW4 -> ROW3
- D_49 pad 1: ROW0 -> ROW3
- D_5 pad 1: ROW4 -> ROW0
- D_50 pad 1: ROW1 -> ROW3
- D_51 pad 1: ROW2 -> ROW3
- D_53 pad 1: ROW4 -> ROW3
- D_54 pad 1: ROW0 -> ROW3
- D_55 pad 1: ROW1 -> ROW4
- D_56 pad 1: ROW2 -> ROW4
- D_57 pad 1: ROW3 -> ROW4
- D_59 pad 1: ROW0 -> ROW4
- D_60 pad 1: ROW1 -> ROW4
- D_61 pad 1: ROW2 -> ROW4
- D_63 pad 1: ROW0 -> ROW4
- D_64 pad 1: ROW1 -> ROW4
- D_66 pad 1: ROW0 -> ROW4
- D_7 pad 1: ROW1 -> ROW0
- D_8 pad 1: ROW2 -> ROW0
- D_9 pad 1: ROW3 -> ROW0
- K_10 pad 1: COL1 -> COL9
- K_11 pad 1: COL2 -> COL10
- K_12 pad 1: COL2 -> COL11
- K_13 pad 1: COL2 -> COL12
- K_14 pad 1: COL2 -> COL13
- K_15 pad 1: COL2 -> COL14
- K_16 pad 1: COL3 -> COL0
- K_17 pad 1: COL3 -> COL1
- K_18 pad 1: COL3 -> COL2
- K_2 pad 1: COL0 -> COL1
- K_20 pad 1: COL3 -> COL4
- K_21 pad 1: COL4 -> COL5
- K_22 pad 1: COL4 -> COL6
- K_23 pad 1: COL4 -> COL7
- K_24 pad 1: COL4 -> COL8
- K_25 pad 1: COL5 -> COL9
- K_26 pad 1: COL5 -> COL10
- K_27 pad 1: COL5 -> COL11
- K_28 pad 1: COL5 -> COL12
- K_29 pad 1: COL5 -> COL13
- K_3 pad 1: COL0 -> COL2
- K_30 pad 1: COL6 -> COL0
- K_31 pad 1: COL6 -> COL1
- K_32 pad 1: COL6 -> COL2
- K_33 pad 1: COL6 -> COL3
- K_34 pad 1: COL6 -> COL4
- K_35 pad 1: COL7 -> COL5
- K_36 pad 1: COL7 -> COL6
- K_38 pad 1: COL7 -> COL8
- K_39 pad 1: COL8 -> COL9
- K_4 pad 1: COL0 -> COL3
- K_40 pad 1: COL8 -> COL10
- K_41 pad 1: COL8 -> COL11
- K_42 pad 1: COL8 -> COL12
- K_43 pad 1: COL8 -> COL0
- K_44 pad 1: COL9 -> COL1
- K_45 pad 1: COL9 -> COL2
- K_46 pad 1: COL9 -> COL3
- K_47 pad 1: COL9 -> COL4
- K_48 pad 1: COL9 -> COL5
- K_49 pad 1: COL10 -> COL6
- K_5 pad 1: COL0 -> COL4
- K_50 pad 1: COL10 -> COL7
- K_51 pad 1: COL10 -> COL8
- K_52 pad 1: COL10 -> COL9
- K_55 pad 1: COL11 -> COL0
- K_56 pad 1: COL11 -> COL1
- K_57 pad 1: COL11 -> COL2
- K_58 pad 1: COL11 -> COL3
- K_59 pad 1: COL12 -> COL4
- K_6 pad 1: COL1 -> COL5
- K_60 pad 1: COL12 -> COL5
- K_61 pad 1: COL12 -> COL6
- K_62 pad 1: COL12 -> COL7
- K_63 pad 1: COL13 -> COL8
- K_64 pad 1: COL13 -> COL9
- K_65 pad 1: COL13 -> COL10
- K_66 pad 1: COL14 -> COL11
- K_7 pad 1: COL1 -> COL6
- K_8 pad 1: COL1 -> COL7
- K_9 pad 1: COL1 -> COL8
- U1 pad 10: ROW2 -> ROW0
- U1 pad 11: ROW3 -> ROW1
- U1 pad 12: ROW4 -> ROW2
- U1 pad 13: unconnected-(U1-PD5_XCK1_CTS-Pad13) -> ROW3
- U1 pad 14: unconnected-(U1-VCC-Pad14) -> Net-(U2-VDD)
- U1 pad 15: unconnected-(U1-GND-Pad15) -> Net-(U2-GND)
- U1 pad 17: unconnected-(U1-PD4_ADC8_ICP1-Pad17) -> ROW4
- U1 pad 2: COL5 -> COL0
- U1 pad 20: COL14 -> COL6
- U1 pad 21: COL13 -> COL7
- U1 pad 22: COL12 -> COL8
- U1 pad 23: COL11 -> COL9
- U1 pad 25: COL9 -> COL11
- U1 pad 26: COL8 -> COL12
- U1 pad 27: COL7 -> COL13
- U1 pad 28: COL6 -> COL14
- U1 pad 3: COL4 -> COL1
- U1 pad 4: COL3 -> COL2
- U1 pad 5: COL2 -> COL3
- U1 pad 6: COL1 -> COL4
- U1 pad 7: COL0 -> Net-(U1-PD0_INT0_SCL_OC0B)
- U1 pad 8: ROW0 -> Net-(U1-PD1_INT1_SDA)
- U1 pad 9: ROW1 -> COL5
Routing:
- net ROW0: track 26.9 -> 472.2 mm
- net ROW1: track 26.9 -> 441.0 mm
- net ROW2: track 26.9 -> 399.8 mm
- net ROW4: track 43.2 -> 398.7 mm
- net ROW3: track 26.9 -> 373.8 mm
- net COL13: track 0.00 -> 308.5 mm
- net COL12: track 0.00 -> 236.4 mm
- net COL11: track 0.00 -> 222.9 mm
- net COL10: track 0.00 -> 193.8 mm
- net COL14: track 0.00 -> 186.5 mm
- net COL9: track 0.00 -> 174.0 mm
- net Net-(D_61-A): track 176.1 -> 11.3 mm
- net Net-(D_66-A): track 177.3 -> 13.8 mm
- net Net-(D_64-A): track 170.1 -> 13.8 mm
- net COL8: track 0.00 -> 156.0 mm
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- removed copper zone on B.Cu, net unconnected-(SW1-Pad2)
- removed copper zone on F.Cu, net unconnected-(SW1-Pad2)
Other:
- board size 363.2 x 95.5 mm -> 366.7 x 95.2 mm
